File: Rev A/crypto_programmer.brd (EAGLE design)
At the start: 50.8 x 50.8 mm, 50 parts, among them J1 10104111-0001LF, J2 M20-9951045, J3 TC2050-IDC-NLFP, J4 DNP, J5 DNP, J6 DNP, U1 ATSAML21E18B-AU, U2 MCP1703AT-3302E/CB, X1 DNP, X2 DNP

Commit message: Updating BOM 2
Parts:
- C6: value 1uF -> 1.0uF
Changed lines of the file:
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@@
 <attribute name="VALUE" x="18.288" y="31.115" size="1.27" layer="28" ratio="11" rot="MR90"/>
 </element>
-<element name="C6" library="rcl" library_urn="urn:adsk.eagle:library:334" package="C0603" value="1uF" x="26.035" y="22.733" smashed="yes" rot="MR0">
+<element name="C6" library="rcl" library_urn="urn:adsk.eagle:library:334" package="C0603" value="1.0uF" x="26.035" y="22.733" smashed="yes" rot="MR0">
 <attribute name="NAME" x="32.385" y="21.717" size="1.27" layer="26" ratio="11" rot="MR0"/>
 <attribute name="VALUE" x="26.67" y="20.828" size="1.27" layer="28" ratio="11" rot="MR0"/>
