File: Rev A/crypto_programmer.sch (EAGLE design)
At the start: 50 parts, among them J1 10104111-0001LF, J2 M20-9951045, J3 TC2050-IDC-NLFP, J4 DNP, J5 DNP, J6 DNP, U1 ATSAML21E18B-AU, U2 MCP1703AT-3302E/CB, X1 DNP, X2 DNP

Commit message: Adding BOM
Parts:
- C14, C15, U2: NOTE Trezor -> (none)
Changed lines of the file:
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@@
 <part name="3.3V3" library="KVB-supply" deviceset="3.3V" device=""/>
 <part name="GND4" library="KVB-supply" deviceset="GND" device=""/>
-<part name="U2" library="KVB-ICs" deviceset="MCP1703AT-3302E/CB" device="">
-<attribute name="NOTE" value="Trezor"/>
-</part>
+<part name="U2" library="KVB-ICs" deviceset="MCP1703AT-3302E/CB" device=""/>
 <part name="GND21" library="KVB-supply" deviceset="GND" device=""/>
-<part name="C14" library="rcl" library_urn="urn:adsk.eagle:library:334" deviceset="C-EU" device="C0603" value="1.0uF">
-<attribute name="NOTE" value="Trezor"/>
-</part>
-<part name="C15" library="rcl" library_urn="urn:adsk.eagle:library:334" deviceset="C-EU" device="C0603" value="1.0uF">
-<attribute name="NOTE" value="Trezor"/>
-</part>
+<part name="C14" library="rcl" library_urn="urn:adsk.eagle:library:334" deviceset="C-EU" device="C0603" value="1.0uF"/>
+<part name="C15" library="rcl" library_urn="urn:adsk.eagle:library:334" deviceset="C-EU" device="C0603" value="1.0uF"/>
 <part name="GND19" library="KVB-supply" deviceset="GND" device=""/>
 <part name="GND23" library="KVB-supply" deviceset="GND" device=""/>
@@
 <attribute name="NAME" x="177.8" y="168.148" size="1.778" layer="95"/>
 <attribute name="VALUE" x="190.5" y="149.86" size="1.778" layer="96"/>
-<attribute name="NOTE" x="177.8" y="167.64" size="1.778" layer="96" display="off"/>
 </instance>
 <instance part="GND21" gate="G$1" x="187.96" y="139.7"/>
-<instance part="C14" gate="G$1" x="162.56" y="157.48">
-<attribute name="NOTE" x="162.56" y="157.48" size="1.778" layer="96" display="off"/>
-</instance>
-<instance part="C15" gate="G$1" x="218.44" y="157.48">
-<attribute name="NOTE" x="218.44" y="157.48" size="1.778" layer="96" display="off"/>
-</instance>
+<instance part="C14" gate="G$1" x="162.56" y="157.48"/>
+<instance part="C15" gate="G$1" x="218.44" y="157.48"/>
 <instance part="GND19" gate="G$1" x="162.56" y="147.32"/>
 <instance part="GND23" gate="G$1" x="218.44" y="147.32"/>

Commit message: Updating BOM 2
Parts:
- C6: value 1uF -> 1.0uF
Changed lines of the file:
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@@
 <part name="C10" library="rcl" library_urn="urn:adsk.eagle:library:334" deviceset="C-EU" device="C0805" value="10uF"/>
 <part name="GND16" library="KVB-supply" deviceset="GND" device=""/>
-<part name="C6" library="rcl" library_urn="urn:adsk.eagle:library:334" deviceset="C-EU" device="C0603" value="1uF"/>
+<part name="C6" library="rcl" library_urn="urn:adsk.eagle:library:334" deviceset="C-EU" device="C0603" value="1.0uF"/>
 <part name="L2" library="KVB-inductors" deviceset="L" device="0603" value="DNP"/>
 <part name="C12" library="rcl" library_urn="urn:adsk.eagle:library:334" deviceset="C-EU" device="C0805" value="10uF"/>
